File: projeto/_autosave-lhc_tijolo32_board.kicad_pcb (KiCad board)
At the start: 2 copper layers, 24 x 84.5 mm, 46 parts, among them J1 USB_A, J2 OLED, J3 JTAG 10pin Connector, J4 CONN_06POLAR, J5 CONN_06POLAR, Q1 MMBT3904, Q2 MMBT3904, SW1 SW_Push, SW2 SW_Push, U1 AP2112K-3.3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

Commit message: Layout updated
Parts:
- moved C8 0.75 mm to (106.4, 56.2), turned to 180 degrees
Connections:
- A1 pad 13: IO27 -> Net-(A1-Pad13)
- A1 pad 3: Net-(A1-Pad3) -> IO27
Routing:
- net ESP_RST: track 23.2 -> 56.9 mm, vias 0 -> 2
- net SDA: track 17.1 -> 48.7 mm, vias 1 -> 2
- net SCL: track 18.7 -> 47.9 mm, vias 1 -> 2
- net IO2: track 0.00 -> 28.1 mm, vias 0 -> 1
- net 5V: track 40.7 -> 66.8 mm, vias 0 -> 4
- net IO5: track 0.00 -> 16.9 mm
- net IO19: track 0.00 -> 13.0 mm
- net GND: track 15.5 -> 20.8 mm
- net IO27: track 0.00 -> 3.90 mm
- net IO12-MTDI: track 11.7 -> 13.6 mm
- net IO35: track 27.7 -> 26.6 mm
- net IO26: track 29.8 -> 28.8 mm
- net IO34: track 23.2 -> 22.5 mm
- net IO32-32kXP: track 18.8 -> 18.9 mm, vias 1 -> 2
