File: projeto/lhc_tijolo32_board.kicad_pcb (KiCad board)
At the start: 2 copper layers, 24 x 84.5 mm, 50 parts, among them J1 USB_A, J2 Conn_01x04, J3 JTAG 10pin Connector, J4 Conn_01x06, J5 Conn_01x06, Q1 MMBT3904, Q2 MMBT3904, SW1 SW_Push, SW2 SW_Push, U1 AP2112K-3.3, U2 CH340G, U3 ESP32-WROOM-32D, U4 AP2112K-3.3, Y1 12MHz 10ppm, Y2 32k 20ppm

Commit message: GERBER atualizado
Other:
- rule pad_to_mask_clearance: 0.051 -> 0

Commit message: #d dos botoes
Changed lines of the file:
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@@
       (outputformat 1)
       (mirror false)
-      (drillshape 1)
+      (drillshape 0)
       (scaleselection 1)
-      (outputdirectory ""))
+      (outputdirectory "output/gerber/"))
   )
   (net 0 "")
@@
       (effects (font (size 0.8 0.8) (thickness 0.12)))
     )
-    (pad 2 smd roundrect (at 1.35 0 90) (size 1.4 1.35) (layers F.Cu F.Paste F.Mask) (roundrect_rratio 0.185185)
-      (net 1 GND))
-    (pad 1 smd roundrect (at -1.35 0 90) (size 1.4 1.35) (layers F.Cu F.Paste F.Mask) (roundrect_rratio 0.185185)
+    (pad 2 smd roundrect (at 1.35 0 90) (size 1.4 1.35) (layers F.Cu F.Paste F.Mask) (roundrect_rratio 0.1851844444444445)
+      (net 1 GND))
+    (pad 1 smd roundrect (at -1.35 0 90) (size 1.4 1.35) (layers F.Cu F.Paste F.Mask) (roundrect_rratio 0.1851844444444445)
       (net 3 +3V3))
     (model ${KISYS3DMOD}/Capacitor_Tantalum_SMD.3dshapes/CP_EIA-3216-12_Kemet-S.wrl
